File: HW/TinyGController_V1.brd (EAGLE design)
At the start: 75 x 100 mm, 52 parts, among them IC1 LM317-3V3, IC2 FT232RL, IC3 7812, IC4 ATXMEGA192A3, Q1 16MHz, T1 IRLML5203TRPBF, X1 PN61729-S

Commit message: Added final V1 and V2 in development
Connections:
- net N$5 renamed FTDI_TXD
- net N$7 renamed FTDI_RXD
Changed lines of the file:
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@@
 <wire x1="5.635" y1="49.54" x2="7.46" y2="49.54" width="0.8" layer="16"/>
 </signal>
-<signal name="N$7">
+<signal name="FTDI_RXD">
 <contactref element="IC2" pad="5"/>
 <contactref element="JP6" pad="8"/>
@@
 <wire x1="24.165" y1="14.375" x2="24.73" y2="13.81" width="0.4" layer="1"/>
 </signal>
-<signal name="N$5">
+<signal name="FTDI_TXD">
 <contactref element="IC2" pad="1"/>
 <contactref element="JP6" pad="6"/>
