File: HW/TinyGController_V1.sch (EAGLE design)
At the start: 52 parts, among them IC1 LM317-3V3, IC2 FT232RL, IC3 7812, IC4 ATXMEGA192A3, Q1 16MHz, T1 IRLML5203TRPBF, X1 PN61729-S

Commit message: Added final V1 and V2 in development
Connections:
- net N$5 renamed FTDI_TXD
- net N$7 renamed FTDI_RXD
Changed lines of the file:
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@@
 </segment>
 </net>
-<net name="N$7" class="0">
+<net name="FTDI_RXD" class="0">
 <segment>
 <pinref part="IC2" gate="G$1" pin="RXD"/>
@@
 </segment>
 </net>
-<net name="N$5" class="0">
+<net name="FTDI_TXD" class="0">
 <segment>
 <wire x1="124.46" y1="152.4" x2="119.38" y2="152.4" width="0.1524" layer="91"/>
